Commit message: moved robot base position

File: abb_irb4600_description/urdf/irb4600_60_205_macro.xacro (robot description, xacro)
@@ -101,5 +101,5 @@
     <!-- joint list -->
     <joint name="${prefix}joint_world" type="fixed">
-      <origin xyz="-8 1 0" rpy="0 0 0"/>
+      <origin xyz="0 0 0" rpy="0 0 0"/>
       <parent link="world"/>
       <child link="${prefix}fake_linear_axis"/>
